File: logger_2G_GSM.brd (EAGLE design)
At the start: 99 x 44.1 mm, 88 parts, among them IC1 LTC4412, J1 POWER_JACKPTH, Q1 FDN360P, Q2 FDN360P, Q3 2N7002PW, Q4 2N7002PW, U1 DS3231MZ/V+T, U2 SIM800H/L, U3 SIM808, X1 32.768, X3 uFL, X4 uFL, X5 1x2, X6 1x2, X7 ANT_2450AT18B100, X8 SIM_LOCKAMPHENOL

Commit message: some progress, keep ATAAMD21G?
Parts:
- removed 3.3_SENSE: LT1461DHS8-5PBF, LTC_By_element14_Batch_1:SOIC127P600X175-8N
- removed ADC1: (no value), adafruit:1X01-CLEANBIG
- removed C1: 10uF, microbuilder:_0805MP
- removed CLOCK, LD0_SD: LP2985, adafruit:SOT23-5L
- removed CLOCK_CIN, SD_CIN, SENSE_CIN: 1uF, rcl:C0603
- removed C_LDO_CLOCK, C_LDO_SD, C_LDO_SENSE: 2.2uF, resistor:C0603
- removed D4, D5, D7, D9: 1N4148, microbuilder:SOD-323
- removed R9: DNP, microbuilder:0603-NO
- removed SJ1: (no value), microbuilder:SOLDERJUMPER_CLOSEDWIRE
- removed TP1: (no value), microbuilder:TESTPOINT_ROUND_1.5MM
- removed U2: SIM800H/L, microbuilder:SIM800L
- removed X5, X6: 1x2, con-molex:87758-0216
- removed X7: ANT_2450AT18B100, microbuilder:ANT_2450AT18B100
- added 3V3: (no value), csandell:6-TMLF
- added CLOCK_CIN1, CLOCK_CIN2, CLOCK_CIN3: 1uF, rcl:C0603
- added RESET1: Reset, SparkFun-Electromechanical:TACTILE-PTH
Connections:
- net RI renamed RING_INDICATOR
- net RTS renamed REQUEST_TO_SEND
- removed net 4_RST: R9.2, U2.49
- removed net 5_UART_DTR: D5.C
- removed net 6_UART_RTS: D4.C
- removed net 7_UART_RI: U2.68
- removed net 8_UART_TXD: U2.32
- removed net 9_UART_RXD: D9.C
- removed net D6-CLOCK_3V3_SWITCH: CLOCK.3
- removed net D8-SD_3V3_SWITCH: LD0_SD.3
- removed net FM_ANT: TP1.P$1, U2.17
- removed net KEY: D7.C, SJ1.2
- removed net MIC1+: U3.P$19
- removed net MIC1-: U3.P$20
- removed net MIC2+: U2.9, X5.1
- removed net MIC2-: U2.10, X5.2
- removed net N$10: ADC1.1, U3.P$23
- removed net N$13: U2.36, X7.FP
- removed net N$16: D7.A, U2.48
- removed net N$18: JP5.VBUS
- removed net N$3: JP5.D+
- removed net N$4: JP5.D-
- removed net SD_CLK: SD.5
- removed net SD_DI: SD.2
- removed net SPEAKER1+: U3.P$21
- removed net SPEAKER1-: U3.P$22
- removed net SPEAKER2+: U2.51, X6.1
- removed net SPEAKER2-: U2.11, X6.2
- removed net UART_DTR: D5.A, U2.69
- removed net UART_RTS: D4.A, U2.33
- new net D6-CLOCK_SD_SWITCH: 3V3.3
- new net VDD_EXT(2.8VOUT): U3.P$7
- net +3V3: now also 3V3.1, CLOCK_CIN2.1; no longer 3.3_SENSE.6, C_LDO_SENSE.2
- net 1.8V: no longer U2.16
- net 2.8V: no longer U2.18, U3.P$7
- net BATTERY_POWER: now also CN1.1, J1.PWR
- net D+: now also JP5.D+
- net D-: now also JP5.D-
- net D4-SENSE_LDO_SWITCH: now also 3V3.4; no longer 3.3_SENSE.3
- net GND: now also 3V3.5, CLOCK_CIN1.2, CLOCK_CIN2.2, CLOCK_CIN3.2, RESET1.1; no longer 3.3_SENSE.4, C1.2, CLOCK.2, CLOCK_CIN.2, C_LDO_CLOCK.1, C_LDO_SD.1, C_LDO_SENSE.1, LD0_SD.2, R9.1, SD_CIN.2, SENSE_CIN.2, SJ1.1, U2.2, U2.35, U2.37, U2.38, U2.39, U2.41, U2.43, U2.44, U2.45, U2.57, U2.58, U2.6, U2.67, U2.71, U2.72, U2.73, U2.76, U2.77, U2.78, U2.79, U2.8, U2.80, U2.81, U2.82, U2.83, U2.84, U2.85, U2.86, U2.87, U2.88
- net GSM_ANT: no longer U2.40
- net MISO: now also SD.7
- net MOSI: now also SD.2
- net NETSTAT: no longer U2.64
- net PWRSTAT: no longer U2.4
- net RESET: now also RESET1.3
- net SCK: now also SD.5
- net SD_DO: no longer SD.7
- net SIMCLK: no longer U2.55
- net SIMDATA: no longer U2.14
- net SIMRST: no longer U2.15
- net UART_RXD: no longer D9.A, U2.31
- net VBAT: no longer U2.1, U2.42
- net VBUS: no longer U2.7
- net VCC: now also 3V3.6, CLOCK_CIN1.1; no longer 3.3_SENSE.2, CLOCK.1, CLOCK_CIN.1, CN1.1, J1.PWR, LD0_SD.1, SD_CIN.1, SENSE_CIN.1
- net VCL: no longer CLOCK.5, C_LDO_CLOCK.2
- net VDD: now also 3V3.2, CLOCK_CIN3.1; no longer C_LDO_SD.2, LD0_SD.5
- net VRTC: no longer C1.1, U2.56
- net VUSB: now also JP5.VBUS
Routing:
- net VCC: track 242.1 -> 0.00 mm, vias 4 -> 0
- net +3V3: track 111.0 -> 0.00 mm, vias 4 -> 0
- net VDD: track 96.0 -> 0.00 mm, vias 5 -> 0
- net RESET: track 86.2 -> 0.00 mm, vias 2 -> 0
- net SDA: track 57.5 -> 0.00 mm, vias 2 -> 0
- net VCL: track 56.8 -> 0.00 mm, vias 4 -> 0
- net 5V: track 53.6 -> 0.00 mm, vias 1 -> 0
- net N$11: track 52.1 -> 0.00 mm, vias 2 -> 0
- net SD_DO: track 51.9 -> 0.00 mm, vias 3 -> 0
- net SCL: track 50.6 -> 0.00 mm, vias 4 -> 0
- net TX-O: track 50.0 -> 0.00 mm, vias 2 -> 0
- net RX-I: track 44.9 -> 0.00 mm, vias 3 -> 0
- net DI: track 41.2 -> 0.00 mm, vias 3 -> 0
- net GND: track 38.0 -> 0.00 mm, vias 36 -> 0
- net SDA_3V3: track 37.2 -> 0.00 mm
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
Commit message: some progress
Parts:
- removed COUT1: 0.1uF, rcl:C0603
- removed LED1: Yellow, SparkFun-LED:LED-0603
- removed LED2: Blue, SparkFun-LED:LED-0603
- removed RESET1: Reset, SparkFun-Electromechanical:TACTILE-PTH
- removed RN1: 1K, resistor-dil:0603-ARC
- removed R_RESET: 10k, rcl:R0603
- added H2: (no value), SparkFun:SCREWTERMINAL-3.5MM-8
- added JP7: (no value), SparkFun-Connectors:SCREWTERMINAL-3.5MM-4
- U$21: value ATSAMD21G18_QFN -> ATSAMD21G18
- X3: value uFL -> GPS
- X4: value uFL -> GSM
- moved CLOCK_CIN3 274.1 mm to (57.5, 33.1), turned to 90 degrees
- moved 3V3 272.5 mm to (59.6, 29.9)
- moved CLOCK_CIN2 270.2 mm to (59.6, 33.1), turned to 90 degrees
- moved CLOCK_CIN1 266.3 mm to (61.6, 33.1), turned to 90 degrees
- moved X8 230.3 mm to (14.9, 22.5)
- moved C3 204.9 mm to (53.7, 31.0)
- moved X1 202.8 mm to (51.9, 33.8)
- moved C4 202.1 mm to (50.7, 31.0), turned to 180 degrees
- moved TP3 201.9 mm to (56.6, 25.9)
- moved TP2 201.3 mm to (56.6, 23.4)
- moved C2 189.2 mm to (56.9, 20.6)
- moved U$21 182.6 mm to (49.1, 21.6), turned to 180 degrees
- moved X4 164.5 mm to (74.5, 29.3), turned to 90 degrees
- moved D3 123.7 mm to (63.1, 14.1), turned to 270 degrees
- moved R6 101.7 mm to (83.1, 20.3), turned to 90 degrees
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Connections:
- removed net 2.8V: R6.2
- removed net AREF: U$21.4
- removed net D0: U$21.16
- removed net D1: U$21.15
- removed net DTR: COUT1.1
- removed net N$20: U$21.48
- removed net N$5: LED2.A, RN1.4
- removed net N$9: LED1.A, RN1.3
- removed net VDD_EXT(2.8VOUT): U3.P$7
- new net N$3: R6.2, U3.P$7
- net +3V3: now also U$21.4
- net A6: now also A6.2, U$21.48; no longer A6.1
- net A7: now also A7.2; no longer A7.1
- net GND: now also A6.1, A7.1; no longer A6.2, A7.2, RESET1.1
- net RESET: no longer COUT1.2, RESET1.3, R_RESET.1
- net RX-I: now also U$21.16
- net TX-O: now also U$21.15
- net VCC: no longer R_RESET.2
- net VUSB: no longer RN1.5, RN1.6
Other:
- board size 99 x 44.1 mm -> 99.1 x 44.1 mm
- board text removed: "Rx"
- board text removed: "Tx"
