File: logger_2G_GSM.sch (EAGLE design)
At the start: 88 parts, among them IC1 LTC4412, J1 POWER_JACKPTH, Q1 FDN360P, Q2 FDN360P, Q3 2N7002PW, Q4 2N7002PW, U1 DS3231MZ/V+T, U2 SIM800H/L, U3 SIM808, X1 32.768, X3 uFL, X4 uFL, X5 1x2, X6 1x2, X7 ANT_2450AT18B100, X8 SIM_LOCKAMPHENOL

Commit message: some progress, keep ATAAMD21G?
Parts:
- removed 3.3_SENSE: LT1461DHS8-5PBF, LTC_By_element14_Batch_1:LT1461DHS8-5PBF
- removed ADC1: (no value), adafruit:PINHD-1X1CB
- removed C1: 10uF, microbuilder:CAP_CERAMIC_0805MP
- removed CLOCK, LD0_SD: LP2985, adafruit:LP298XS
- removed CLOCK_CIN, SD_CIN, SENSE_CIN: 1uF, rcl:C-EUC0603
- removed C_LDO_CLOCK, C_LDO_SD, C_LDO_SENSE: 2.2uF, resistor:C-EUC0603
- removed D4, D5, D7, D9: 1N4148, microbuilder:DIODESOD-323
- removed R9: DNP, microbuilder:RESISTOR_0603_NOOUT
- removed SJ1: (no value), microbuilder:SOLDERJUMPER_CLOSED
- removed TP1: (no value), microbuilder:TESTPOINTROUND1.5MM
- removed U2: SIM800H/L, microbuilder:GSM_SIM800L
- removed X5, X6: 1x2, con-molex:87758-0216
- removed X7: ANT_2450AT18B100, microbuilder:ANTENNA_JOHANSON_2450AT18B100
- added 3V3: (no value), csandell:MIC5380
- added CLOCK_CIN1, CLOCK_CIN2, CLOCK_CIN3: 1uF, rcl:C-EUC0603
- added RESET1: Reset, SparkFun-Electromechanical:SWITCH-MOMENTARY-2PTH
Connections:
- net RI renamed RING_INDICATOR
- net RTS renamed REQUEST_TO_SEND
- removed net 4_RST: R9.2, U2.RESET
- removed net 5_UART_DTR: D5.C
- removed net 6_UART_RTS: D4.C
- removed net 7_UART_RI: U2.UART_RI
- removed net 8_UART_TXD: U2.UART_TXD
- removed net 9_UART_RXD: D9.C
- removed net D6-CLOCK_3V3_SWITCH: CLOCK.EN
- removed net D8-SD_3V3_SWITCH: LD0_SD.EN
- removed net FM_ANT: TP1.P$1, U2.FM_ANT_P
- removed net KEY: D7.C, SJ1.2
- removed net MIC1+: U3.MIC1P
- removed net MIC1-: U3.MIC1N
- removed net MIC2+: U2.MIC2P, X5-1.S
- removed net MIC2-: U2.MIC2N, X5-2.S
- removed net N$10: ADC1.1, U3.ADC1
- removed net N$13: U2.NC, X7.P$1
- removed net N$16: D7.A, U2.PWRKEY
- removed net N$18: JP5.VBUS
- removed net N$3: JP5.D+
- removed net N$4: JP5.D-
- removed net SD_CLK: SD.SCLK
- removed net SD_DI: SD.DATA_IN
- removed net SPEAKER1+: U3.SPK1P
- removed net SPEAKER1-: U3.SPK1N
- removed net SPEAKER2+: U2.SPK2P/8Ω, X6-1.S
- removed net SPEAKER2-: U2.SPK2N, X6-2.S
- removed net UART_DTR: D5.A, U2.UART_DTR
- removed net UART_RTS: D4.A, U2.UART_RTS
- new net D6-CLOCK_SD_SWITCH: 3V3.EN2
- net +3V3: now also 3V3.VOUT1, CLOCK_CIN2.1; no longer 3.3_SENSE.VOUT, C_LDO_SENSE.2
- net 1.8V: no longer U2.VSIM
- net 2.8V: no longer U2.VEXT, U3.VDD_EXT(2.8VOUT)
- net BATTERY_POWER: now also CN1.2, J1.PWR
- net D+: now also JP5.D+
- net D-: now also JP5.D-
- net D4-SENSE_LDO_SWITCH: now also 3V3.EN1; no longer 3.3_SENSE.~SHDN
- net GND: now also 3V3.GND, CLOCK_CIN1.2, CLOCK_CIN2.2, CLOCK_CIN3.2, RESET1.1; no longer 3.3_SENSE.GND, C1.2, CLOCK.GND, CLOCK_CIN.2, C_LDO_CLOCK.1, C_LDO_SD.1, C_LDO_SENSE.1, LD0_SD.GND, R9.1, SD_CIN.2, SENSE_CIN.2, SJ1.1, U2.FM_ANT_N, U2.GND
- net GSM_ANT: no longer U2.ANT
- net MISO: now also SD.DATA_OUT
- net MOSI: now also SD.DATA_IN
- net NETSTAT: no longer U2.NETLIGHT
- net PWRSTAT: no longer U2.STATUS
- net RESET: now also RESET1.2
- net SCK: now also SD.SCLK
- net SD_DO: no longer SD.DATA_OUT
- net SIMCLK: no longer U2.SIM_CLK
- net SIMDATA: no longer U2.SIM_DATA
- net SIMRST: no longer U2.SIM_RST
- net UART_RXD: no longer D9.A, U2.UART_RXD
- net VBAT: no longer U2.VBAT
- net VCC: now also 3V3.VIN, CLOCK_CIN1.1; no longer 3.3_SENSE.VIN, CLOCK.VIN, CLOCK_CIN.1, CN1.2, J1.PWR, LD0_SD.VIN, SD_CIN.1, SENSE_CIN.1
- net VCL: no longer CLOCK.VOUT, C_LDO_CLOCK.2
- net VDD: now also 3V3.VOUT2, CLOCK_CIN3.1; no longer C_LDO_SD.2, LD0_SD.VOUT
- net VRTC: no longer C1.1, U2.VRTC
- net VUSB: now also JP5.VBUS
Other:
- note added: "CELLULAR COMMUNICATION"
- note added: "SD CARD"
- note added: "SIM CARD"
- note removed: "3V3 = Sensor 3V3"
- note removed: "SD CARD AND LEVEL SHIFTER"
- note removed: "VCL = CLOCK 3V3"
- note removed: "VDD = SD3V3"
- moved on the sheet: 5V_CHARGE_PUMP, C14A, C14B, C9, CN1, COUT, COUT1, C_BOOST_1, C_BOOST_2, C_BOOST_3, D3, IC1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

Commit message: some progress
Parts:
- removed COUT1: 0.1uF, rcl:C-EUC0603
- removed LED1: Yellow, SparkFun-LED:LED0603
- removed LED2: Blue, SparkFun-LED:LED0603
- removed RESET1: Reset, SparkFun-Electromechanical:SWITCH-MOMENTARY-2PTH
- removed RN1: 1K, resistor-dil:4R-N0603-ARC
- removed R_RESET: 10k, rcl:R-US_R0603
- added H2: (no value), SparkFun:M083.5MM-8
- added JP7: (no value), SparkFun-Connectors:M04SCREW
- U$21: value ATSAMD21G18_QFN -> ATSAMD21G18
- X3: value uFL -> GPS
- X4: value uFL -> GSM
Connections:
- removed net 2.8V: R6.2
- removed net AREF: U$21.PA03/EINT3/VREFA/AIN1
- removed net D0: U$21.PA11/I11/AIN19/SERCOM0+2.3/I2SF0
- removed net D1: U$21.PA10/I10/AIN18/SERCOM0+2.2/I2SCK
- removed net DTR: COUT1.1
- removed net N$20: U$21.PB03/I3/AIN11/SERCOM5.1
- removed net N$5: LED2.A, RN1D.1
- removed net N$9: LED1.A, RN1C.1
- new net N$3: R6.2, U3.VDD_EXT(2.8VOUT)
- net +3V3: now also U$21.PA03/EINT3/VREFA/AIN1
- net A6: now also A6.2, U$21.PB03/I3/AIN11/SERCOM5.1; no longer A6.1
- net A7: now also A7.2; no longer A7.1
- net GND: now also A6.1, A7.1; no longer A6.2, A7.2, RESET1.1
- net RESET: no longer COUT1.2, RESET1.2, R_RESET.1
- net RX-I: now also U$21.PA11/I11/AIN19/SERCOM0+2.3/I2SF0
- net TX-O: now also U$21.PA10/I10/AIN18/SERCOM0+2.2/I2SCK
- net VCC: no longer R_RESET.2
- net VUSB: no longer RN1C.2, RN1D.2
Other:
- moved on the sheet: A6, A7, RESET
